Commit message: enforced a fixed frame for robot + increased gripper spacing

File: youbot_description/robots/youbot_with_cam3d.urdf.xacro (robot description, xacro)
@@ -56,3 +56,8 @@
     <origin xyz="0 0 0.49" rpy="0 0 0" />
   </xacro:asus_xtion_camera>
+  <link name="world"/>
+  <joint name="grouding" type="fixed">
+    <parent link="world"/>
+    <child link="base_footprint"/>
+  </joint>
 </robot>

File: youbot_description/urdf/youbot_gripper/gripper.urdf.xacro (robot description, xacro)
@@ -36,5 +36,5 @@
 		</link>
 		<joint name="${name}_finger_joint_l" type="prismatic">
-			<origin xyz="0.004 0.008 0.046" rpy="0 0 ${M_PI}" />
+			<origin xyz="0.004 0.02 0.046" rpy="0 0 ${M_PI}" />
 			<parent link="${name}_palm_link"/>
 			<child link="${name}_finger_link_l"/>
@@ -66,5 +66,5 @@
 		</link>
                <joint name="${name}_finger_joint_r" type="prismatic">
-			<origin xyz="0.004 -0.008 0.046" rpy="0 0 0" />
+			<origin xyz="0.004 -0.02 0.046" rpy="0 0 0" />
 			<parent link="${name}_palm_link"/>
 			<child link="${name}_finger_link_r"/>

Commit message: changes to support Xtion camera on the arm - config files with position - moveit planning config file - disable collisions in motion planning with camera and arm link

File: youbot_description/robots/youbot_with_cam3d.urdf.xacro (robot description, xacro)
@@ -23,6 +23,4 @@
   <xacro:include filename="$(find youbot_description)/urdf/sensors/hokuyo_urg04_laser.urdf.xacro"/>
   <xacro:include filename="$(find youbot_description)/urdf/sensors/asus_xtion_camera.urdf.xacro"/>
-  <!-- sensor tower -->
-  <xacro:include filename="$(find youbot_description)/urdf/misc/camera_tower.urdf.xacro"/>
   <!-- Now we can start using the macros xacro:included above to define the actual youbot -->
   <!-- The first use of a macro.  This one was defined in base.urdf.xacro above.
@@ -48,11 +46,7 @@
     <origin xyz="0.3 0 -0.03" rpy="0 0 0"/>
   </xacro:hokuyo_urg04_laser>
-  <!-- camera tower -->
-  <xacro:camera_tower name="camera_tower" parent="plate_link">
-    <origin xyz="-0.11 0.0 0.03" rpy="0 0 0" />
-  </xacro:camera_tower>
   <!-- 3D camera on tower -->
-  <xacro:asus_xtion_camera name="arm_cam3d" parent="camera_tower_link" tilt="0.5">
-    <origin xyz="0 0 0.49" rpy="0 0 0" />
+  <xacro:asus_xtion_camera name="arm_cam3d" parent="arm_link_4" tilt="0.0">
+    <origin xyz="0.025 0 0.045" rpy="0 -1.5707 3.14159" />
   </xacro:asus_xtion_camera>
   <link name="world"/>
