Commit message: changed the camera placing on the arm

File: youbot_description/robots/youbot.urdf.xacro (robot description, xacro)
@@ -22,4 +22,5 @@
   <!-- sensors -->
   <xacro:include filename="$(find youbot_description)/urdf/sensors/hokuyo_urg04_laser.urdf.xacro"/>
+	<xacro:include filename="$(find youbot_description)/urdf/sensors/asus_xtion_camera.urdf.xacro"/>
   <!-- Now we can start using the macros xacro:included above to define the actual youbot -->
   <!-- The first use of a macro.  This one was defined in base.urdf.xacro above.

File: youbot_description/urdf/youbot_gripper/gripper.urdf.xacro (robot description, xacro)
@@ -95,4 +95,8 @@
 			</collision>
 		</link>
+	  <!-- 3D camera on tower -->
+	  <xacro:asus_xtion_camera name="arm_cam3d" parent="${name}_palm_link" tilt="0.0">
+	    <origin xyz="0.025 0 0.045" rpy="0 -1.5707 3.14159" />
+	  </xacro:asus_xtion_camera>
 		<!-- extensions -->
 		<xacro:youbot_gripper_gazebo name="${name}" />

Commit message: added friction to task world object for better simulation - added grounding of youbot for simulation purposes

File: youbot_description/robots/youbot.urdf.xacro (robot description, xacro)
@@ -45,3 +45,8 @@
     <origin xyz="0.3 0 -0.03" rpy="0 0 0"/>
   </xacro:hokuyo_urg04_laser>
+  <link name="world"/>
+  <joint name="grouding" type="fixed">
+    <parent link="world"/>
+    <child link="base_footprint"/>
+  </joint>
 </robot>

File: youbot_simulation/youbot_gazebo_worlds/urdf/picknplace.urdf (robot description, URDF)
Before this commit: robot arena, 1 links, 0 joints
Links:
- link box1: mass 0.01 -> 0.00001
