Commit message: positioning of camera on gripper - disbaled collisions for necessary links for MoveIt - added magic line to kinematics.yaml - urdf specs

File: youbot_description/urdf/youbot_gripper/gripper.urdf.xacro (robot description, xacro)
@@ -97,5 +97,5 @@
 	  <!-- 3D camera on tower -->
 	  <xacro:asus_xtion_camera name="arm_cam3d" parent="${name}_palm_link" tilt="0.0">
-	    <origin xyz="0.025 0 0.045" rpy="0 -1.5707 3.14159" />
+	    <origin xyz="0.01972 -0.0342 0.0459" rpy="0.02 0.0076 3.094" />
 	  </xacro:asus_xtion_camera>
 		<!-- extensions -->

Commit message: better placing for camera after gazebo verification - disabled some collisions that were preventing motion planning

File: youbot_description/urdf/youbot_gripper/gripper.urdf.xacro (robot description, xacro)
@@ -97,5 +97,5 @@
 	  <!-- 3D camera on tower -->
 	  <xacro:asus_xtion_camera name="arm_cam3d" parent="${name}_palm_link" tilt="0.0">
-	    <origin xyz="0.01972 -0.0342 0.0459" rpy="0.02 0.0076 3.094" />
+	    <origin xyz="0.025 0.0 -0.02" rpy="0 -1.5707 3.14159" />
 	  </xacro:asus_xtion_camera>
 		<!-- extensions -->

Commit message: changed camera orientation to point backwards - allows for more range in object detection

File: youbot_description/urdf/youbot_gripper/gripper.urdf.xacro (robot description, xacro)
@@ -97,5 +97,5 @@
 	  <!-- 3D camera on tower -->
 	  <xacro:asus_xtion_camera name="arm_cam3d" parent="${name}_palm_link" tilt="0.0">
-	    <origin xyz="0.025 0.0 -0.02" rpy="0 -1.5707 3.14159" />
+	    <origin xyz="0.025 0.0 0.0" rpy="0.0 1.5707 0.0" />
 	  </xacro:asus_xtion_camera>
 		<!-- extensions -->

Commit message: fixed offset to reflect new camera mount

File: youbot_description/urdf/youbot_gripper/gripper.urdf.xacro (robot description, xacro)
@@ -97,5 +97,5 @@
 	  <!-- 3D camera on tower -->
 	  <xacro:asus_xtion_camera name="arm_cam3d" parent="${name}_palm_link" tilt="0.0">
-	    <origin xyz="0.025 0.0 0.0" rpy="0.0 1.5707 0.0" />
+	    <origin xyz="0.04 0.0 0.025" rpy="0.0 1.5707 0.0" />
 	  </xacro:asus_xtion_camera>
 		<!-- extensions -->

Commit message: URDF edit from silva

File: youbot_description/urdf/youbot_gripper/gripper.urdf.xacro (robot description, xacro)
@@ -97,5 +97,5 @@
 	  <!-- 3D camera on tower -->
 	  <xacro:asus_xtion_camera name="arm_cam3d" parent="${name}_palm_link" tilt="0.0">
-	    <origin xyz="0.04 0.0 0.025" rpy="0.0 1.5707 0.0" />
+	    <origin xyz="0.04 -0.02 0.025" rpy="0.0 1.5707 0.0" />
 	  </xacro:asus_xtion_camera>
 		<!-- extensions -->
